File: board/board.kicad_pcb (KiCad board)
At the start: 2 copper layers, 53.8 x 63.8 mm, 36 parts, among them J1 Conn_01x07_Pin, J2 Conn_01x06_Pin, J3 Conn_01x10_Pin, J4 Conn_01x08_Pin, J5 Conn_01x04_Socket, J6 Conn_01x04_Socket, J7 RJ45_Hanrun_HR911105A_Horizon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, J8 Conn_01x02_Pin, U1 7414, U2 AMS1117-3.3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

Commit message: Small changes prior to ordering
Parts:
- added C7: 100n, Capacitor_SMD:C_0603_1608Metric, F.Cu at (117.4, 103.2)
Routing:
- net +5V: track 83.6 -> 85.6 mm
- net GND: track 32.1 -> 33.3 mm, vias 21 -> 22
Other:
- board text added: "capybara"
