File: board/board.kicad_pcb (KiCad board)
At the start: 2 copper layers, 53.8 x 63.8 mm, 37 parts, among them J1 Conn_01x07_Pin, J2 Conn_01x06_Pin, J3 Conn_01x10_Pin, J4 Conn_01x08_Pin, J5 Conn_01x04_Socket, J6 Conn_01x04_Socket, J7 RJ45_Hanrun_HR911105A_Horizon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, J8 Conn_01x02_Pin, U1 7414, U2 AMS1117-3.3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

Commit message: Removal of C4 and C5 from Ethernet rx lines
Parts:
- removed C4, C5: 6.8n, Capacitor_SMD:C_0603_1608Metric
- moved R2 0.45 mm to (95.4, 66.8), turned to -90 degrees
Connections:
- J7 pad 3: Net-(J7-RD+) -> RXIP
- J7 pad 6: Net-(J7-RD-) -> RXIN
Routing:
- net RXIN: track 7.87 -> 16.6 mm
- net RXIP: track 6.93 -> 15.6 mm
- net Net-(J7-RD+): track 7.72 -> 0.00 mm
- net Net-(J7-RD-): track 5.43 -> 0.00 mm
- net Net-(J7-RCT): track 15.0 -> 13.5 mm
