File: board/board.kicad_sch (KiCad schematic)
At the start: 36 parts, among them J1 Conn_01x07_Pin, J2 Conn_01x06_Pin, J3 Conn_01x10_Pin, J4 Conn_01x08_Pin, J5 Conn_01x04_Socket, J6 Conn_01x04_Socket, J7 RJ45_Hanrun_HR911105A_Horizon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, J8 Conn_01x02_Pin, U1 7414, U2 AMS1117-3.3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

Commit message: Small changes prior to ordering
Parts:
- added C7: 100n, Capacitor_SMD:C_0603_1608Metric, symbol Device:C
Connections:
- net +5V: now also C7.1
- net GND: now also C7.2
Changed lines of the file:
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@@
 	)
 	(junction
+		(at 38.1 101.6)
+		(diameter 0)
+		(color 0 0 0 0)
+	)
+	(junction
 		(at 21.59 247.65)
 		(diameter 0)
@@
 	)
 	(junction
-		(at 226.06 93.98)
-		(diameter 0)
-		(color 0 0 0 0)
-	)
-	(junction
 		(at 171.45 240.03)
 		(diameter 0)
@@
 	)
 	(junction
+		(at 36.83 134.62)
+		(diameter 0)
+		(color 0 0 0 0)
+	)
+	(junction
 		(at 171.45 232.41)
 		(diameter 0)
@@
 	(wire
 		(pts
-			(xy 53.34 62.23) (xy 53.34 67.31)
+			(xy 236.22 90.17) (xy 236.22 96.52)
 		)
 		(stroke
@@
 	(wire
 		(pts
-			(xy 236.22 90.17) (xy 236.22 96.52)
+			(xy 237.49 246.38) (xy 237.49 248.92)
 		)
 		(stroke
@@
 	(wire
 		(pts
-			(xy 237.49 246.38) (xy 237.49 248.92)
+			(xy 53.34 129.54) (xy 53.34 134.62)
 		)
 		(stroke
@@
 	(wire
 		(pts
-			(xy 53.34 129.54) (xy 53.34 134.62)
+			(xy 92.71 134.62) (xy 109.22 134.62)
 		)
 		(stroke
@@
 	(wire
 		(pts
-			(xy 92.71 134.62) (xy 109.22 134.62)
+			(xy 128.27 190.5) (xy 135.89 190.5)
 		)
 		(stroke
@@
 	(wire
 		(pts
-			(xy 128.27 190.5) (xy 135.89 190.5)
+			(xy 53.34 91.44) (xy 92.71 91.44)
 		)
 		(stroke
@@
 	(wire
 		(pts
-			(xy 53.34 91.44) (xy 92.71 91.44)
+			(xy 33.02 247.65) (xy 36.83 247.65)
 		)
 		(stroke
@@
 	(wire
 		(pts
-			(xy 33.02 247.65) (xy 36.83 247.65)
+			(xy 24.13 101.6) (xy 24.13 113.03)
 		)
 		(stroke
@@
 	(wire
 		(pts
+			(xy 38.1 101.6) (xy 24.13 101.6)
+		)
+		(stroke
+			(width 0)
+			(type default)
+		)
+	)
+	(wire
+		(pts
 			(xy 135.89 205.74) (xy 143.51 205.74)
 		)
@@
 	(wire
 		(pts
-			(xy 39.37 62.23) (xy 53.34 62.23)
-		)
-		(stroke
-			(width 0)
-			(type default)
-		)
-	)
-	(wire
-		(pts
 			(xy 171.45 212.09) (xy 166.37 212.09)
 		)
@@
 	(wire
 		(pts
-			(xy 226.06 93.98) (xy 226.06 97.79)
+			(xy 162.56 212.09) (xy 162.56 214.63)
 		)
 		(stroke
@@
 	(wire
 		(pts
-			(xy 162.56 212.09) (xy 162.56 214.63)
+			(xy 171.45 251.46) (xy 171.45 254)
 		)
 		(stroke
@@
 	(wire
 		(pts
-			(xy 171.45 251.46) (xy 171.45 254)
+			(xy 74.93 189.23) (xy 80.01 189.23)
 		)
 		(stroke
@@
 	(wire
 		(pts
-			(xy 74.93 189.23) (xy 80.01 189.23)
+			(xy 109.22 240.03) (xy 109.22 248.92)
 		)
 		(stroke
@@
 	(wire
 		(pts
-			(xy 109.22 240.03) (xy 109.22 248.92)
+			(xy 24.13 120.65) (xy 24.13 134.62)
 		)
 		(stroke
@@
 	(wire
 		(pts
+			(xy 53.34 62.23) (xy 92.71 62.23)
+		)
+		(stroke
+			(width 0)
+			(type default)
+		)
+	)
+	(wire
+		(pts
 			(xy 190.5 214.63) (xy 190.5 212.09)
 		)
@@
 	(wire
 		(pts
-			(xy 171.45 254) (xy 167.64 254)
+			(xy 36.83 134.62) (xy 53.34 134.62)
 		)
 		(stroke
@@
 	(wire
 		(pts
-			(xy 171.45 71.12) (xy 177.8 71.12)
+			(xy 171.45 254) (xy 167.64 254)
 		)
 		(stroke
@@
 	(wire
 		(pts
-			(xy 53.34 22.86) (xy 39.37 22.86)
+			(xy 171.45 71.12) (xy 177.8 71.12)
 		)
 		(stroke
@@
 	(wire
 		(pts
-			(xy 135.89 190.5) (xy 143.51 190.5)
+			(xy 53.34 22.86) (xy 39.37 22.86)
 		)
 		(stroke
@@
 	(wire
 		(pts
-			(xy 189.23 234.95) (xy 201.93 234.95)
+			(xy 135.89 190.5) (xy 143.51 190.5)
 		)
 		(stroke
@@
 	(wire
 		(pts
-			(xy 80.01 189.23) (xy 80.01 191.77)
+			(xy 189.23 234.95) (xy 201.93 234.95)
 		)
 		(stroke
@@
 	(wire
 		(pts
-			(xy 113.03 190.5) (xy 120.65 190.5)
+			(xy 80.01 189.23) (xy 80.01 191.77)
 		)
 		(stroke
@@
 	(wire
 		(pts
-			(xy 66.04 39.37) (xy 73.66 39.37)
+			(xy 113.03 190.5) (xy 120.65 190.5)
 		)
 		(stroke
@@
 	(wire
 		(pts
-			(xy 36.83 134.62) (xy 53.34 134.62)
+			(xy 66.04 39.37) (xy 73.66 39.37)
 		)
 		(stroke
@@
 	(wire
 		(pts
-			(xy 53.34 62.23) (xy 92.71 62.23)
+			(xy 39.37 62.23) (xy 53.34 62.23)
 		)
 		(stroke
@@
 	(wire
 		(pts
-			(xy 226.06 90.17) (xy 226.06 93.98)
+			(xy 226.06 90.17) (xy 226.06 97.79)
 		)
 		(stroke
@@
 	(wire
 		(pts
-			(xy 66.04 119.38) (xy 80.01 119.38)
+			(xy 24.13 134.62) (xy 36.83 134.62)
 		)
 		(stroke
@@
 	(wire
 		(pts
-			(xy 92.71 109.22) (xy 92.71 101.6)
+			(xy 66.04 119.38) (xy 80.01 119.38)
 		)
 		(stroke
@@
 	(wire
 		(pts
-			(xy 232.41 245.11) (xy 232.41 246.38)
+			(xy 92.71 109.22) (xy 92.71 101.6)
 		)
 		(stroke
@@
 	(wire
 		(pts
-			(xy 160.02 234.95) (xy 162.56 234.95)
+			(xy 232.41 245.11) (xy 232.41 246.38)
 		)
 		(stroke
@@
 	(wire
 		(pts
-			(xy 219.71 93.98) (xy 226.06 93.98)
+			(xy 160.02 234.95) (xy 162.56 234.95)
 		)
 		(stroke
@@
 	(wire
 		(pts
+			(xy 53.34 62.23) (xy 53.34 67.31)
+		)
+		(stroke
+			(width 0)
+			(type default)
+		)
+	)
+	(wire
+		(pts
 			(xy 236.22 109.22) (xy 236.22 104.14)
 		)
@@
 		)
 	)
-	(global_label "5V"
+	(global_label "+5V"
 		(shape input)
 		(at 148.59 85.09 0)
@@
 		)
 		(property "Intersheetrefs" "${INTERSHEET_REFS}"
-			(at 153.8733 85.09 0)
+			(at 155.4457 85.09 0)
 			(effects
 				(font
@@
 		)
 	)
-	(global_label "5V"
-		(shape input)
-		(at 219.71 93.98 180)
-		(fields_autoplaced yes)
-		(effects
-			(font
-				(size 1.27 1.27)
-			)
-			(justify right)
-		)
-		(property "Intersheetrefs" "${INTERSHEET_REFS}"
-			(at 214.4267 93.98 0)
-			(effects
-				(font
-					(size 1.27 1.27)
-				)
-				(justify right)
-				(hide yes)
-			)
-		)
-	)
 	(global_label "+5V"
 		(shape input)
@@
 					(unit 1)
 				)
+			)
+		)
+	)
+	(symbol
+		(lib_id "Device:C")
+		(at 24.13 116.84 0)
+		(unit 1)
+		(exclude_from_sim no)
+		(in_bom yes)
+		(on_board yes)
+		(dnp no)
+		(fields_autoplaced yes)
+		(property "Reference" "C7"
+			(at 27.94 115.5699 0)
+			(effects
+				(font
+					(size 1.27 1.27)
+				)
+				(justify left)
+			)
+		)
+		(property "Value" "100n	"
+			(at 27.94 118.1099 0)
+			(effects
+				(font
+					(size 1.27 1.27)
+				)
+				(justify left)
+			)
+		)
+		(property "Footprint" "Capacitor_SMD:C_0603_1608Metric"
+			(at 25.0952 120.65 0)
+			(effects
+				(font
+					(size 1.27 1.27)
+				)
+				(hide yes)
+			)
+		)
+		(property "Datasheet" "~"
+			(at 24.13 116.84 0)
+			(effects
+				(font
+					(size 1.27 1.27)
+				)
+				(hide yes)
+			)
+		)
+		(property "Description" "Unpolarized capacitor"
+			(at 24.13 116.84 0)
+			(effects
+				(font
+					(size 1.27 1.27)
+				)
+				(hide yes)
+			)
+		)
+		(pin "2"
+		)
+		(pin "1"
+		)
+		(instances
+			(project "board"
+				(path "/22fdffbc-e246-4dea-9283-18974779b154"
+					(reference "C7")
+					(unit 1)
+				)
